File: schematic/smdrv/sm-driver.kicad_pcb (KiCad board)
At the start: 2 copper layers, 34 parts, among them U1 L297, U2 L298N

Commit message: Small update
Parts:
- U2: moved to F.Cu
- moved LED2 236.2 mm to (236.2, 271.8), turned to 0 degrees
- moved LED1 233.9 mm to (200.0, 267.3)
- moved R1 215.7 mm to (244.5, 255.3), turned to 0 degrees
- moved PIN5 212.4 mm to (257.2, 248.9)
- moved R2 209.1 mm to (213.4, 247.7)
- moved D9 197.5 mm to (255.3, 265.4)
- moved R4 186.0 mm to (183.5, 268.6)
- moved PIN7 179.1 mm to (209.6, 276.2)
- moved R6 178.8 mm to (248.9, 240.0)
- moved PIN4 178.6 mm to (194.9, 251.5), turned to 0 degrees
- moved R5 173.1 mm to (230.5, 261.6)
- moved PIN11 172.0 mm to (221.0, 271.8)
- moved C1 170.5 mm to (214.0, 259.1)
- moved PIN3 148.5 mm to (170.8, 238.8)
- moved PIN10 145.8 mm to (245.1, 228.0)
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Connections:
- D2 pad 1: N-0000022 (its old number) -> GND
- D4 pad 1: N-0000022 (its old number) -> GND
- D6 pad 1: N-0000022 (its old number) -> GND
- D8 pad 1: N-0000022 (its old number) -> GND
- PIN2 pad 1: +5V -> GND
- PIN2 pad 2: GND -> +5V
Routing:
- net +36V: track 179.4 -> 57.5 mm
- net GND: track 102.3 -> 24.3 mm
- net N-0000025: track 57.9 -> 132.1 mm
- net +5V: track 65.4 -> 0.00 mm
- net N-0000022 (its old number): track 65.4 -> 0.00 mm
- net N-000006: track 99.1 -> 36.2 mm
- net N-0000027: track 34.5 -> 0.00 mm
- net N-0000026: track 22.4 -> 0.00 mm
- net N-0000020: track 20.0 -> 0.00 mm
- net N-0000012: track 18.9 -> 0.00 mm
- net N-0000014: track 18.9 -> 0.00 mm
- net N-0000013: track 14.4 -> 0.00 mm
- net N-0000021: track 14.4 -> 0.00 mm
- net N-0000024: track 59.2 -> 45.5 mm
- net N-0000015: track 13.3 -> 0.00 mm
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Other:
- net class Default: via_dia 0.889 -> 1.8; via_drill 0.635 -> 1.1
- rule trace_min: 0.254 -> 0.3
- rule via_min_drill: 0.508 -> 1.1
- rule via_min_size: 0.889 -> 1.8

Commit message: Routing in progress
Parts:
- moved PIN11 117.0 mm to (175.9, 163.8), turned to 270 degrees
- moved PIN7 110.0 mm to (175.9, 171.4), turned to 270 degrees
- moved PIN4 103.0 mm to (247.0, 162.6), turned to 90 degrees
- moved PIN1 81.4 mm to (175.9, 174.0), turned to 270 degrees
- moved PIN2 76.7 mm to (175.9, 166.4), turned to 270 degrees
- moved PIN3 62.4 mm to (175.9, 176.5), turned to 270 degrees
- moved PIN10 59.7 mm to (185.4, 229.2)
- moved PIN6 54.3 mm to (175.9, 184.2), turned to 270 degrees
- moved U1 15.7 mm to (194.9, 184.2)
Connections:
- PIN2 pad 1: GND -> +5V
- PIN2 pad 2: +5V -> GND
Routing:
- net GND: track 24.3 -> 72.7 mm, vias 0 -> 2
- net N-0000011: track 0.00 -> 31.8 mm
- net N-0000010: track 0.00 -> 21.2 mm
- net N-0000026: track 0.00 -> 20.1 mm
- net +5V: track 0.00 -> 12.5 mm
- net N-0000027: track 0.00 -> 11.4 mm
- net N-0000021: track 0.00 -> 11.4 mm
- net N-0000018: track 0.00 -> 11.4 mm
- net N-0000017: track 0.00 -> 11.4 mm
