File: schematic/smdrv/sm-driver.kicad_pcb (KiCad board)
At the start: 2 copper layers, 75.6 x 80 mm, 35 parts, among them U1 L297, U2 L298N

Commit message: smdrv-rev.4-1 release
Parts:
- added R8: 0, RES_1206, F.Cu at (227.3, 141.0)
- moved C2 1.91 mm to (179.7, 156.2)
- moved PIN8 0.64 mm to (197.5, 109.2)
- moved PIN9 0.64 mm to (238.1, 109.2)
- moved PIN4 0.63 mm to (246.4, 162.6)
Connections:
- PIN11 pad 1: N-0000028 (its old number) -> N-0000026
- R1 pad 1: N-0000028 (its old number) -> N-000005
- U1 pad 10: N-0000028 (its old number) -> N-0000026
Routing:
- net N-0000025: track 191.1 -> 66.9 mm
- net N-000005: track 0.00 -> 90.5 mm
- net N-0000026: track 0.00 -> 76.8 mm
- net +5V: track 189.2 -> 136.4 mm, vias 3 -> 2
- net N-0000028 (its old number): track 50.9 -> 0.00 mm, vias 2 -> 0
- net GND: track 338.5 -> 300.4 mm, vias 3 -> 0
- net N-0000030: track 70.1 -> 76.8 mm
- net N-0000023: track 75.0 -> 80.7 mm
- net N-0000017: track 64.2 -> 69.7 mm
- net +36V: track 149.4 -> 145.2 mm
- net N-0000020: track 94.2 -> 96.9 mm
- net N-0000024: track 102.2 -> 99.8 mm
- net N-0000013: track 26.2 -> 25.2 mm
- net N-000008: track 19.3 -> 19.8 mm
Other:
- outline, holes or cut-outs redrawn
- net class Default: via_dia 1.8 -> 1.7; via_drill 1.1 -> 1.2
- rule via_min_drill: 1.1 -> 1.2
- rule via_min_size: 1.8 -> 1.7
- board text added: "stepper motor driver open3dp-mk.1-rev.4-1 Ivanov S., 2013"
- board text removed: "stepper motor driver open3dp-mk.1-rev.4 Ivanov S., 2013"
