File: schematic/smdrv/sm-driver.kicad_pcb (KiCad board)
At the start: 2 copper layers, 35 parts, among them U1 L297, U2 L298N

Commit message: Prepare motor driver mk.1 for prototyping.
Parts:
- removed C1, C3: 470n, C_CERAM
- removed C2, C4: 100n, C_CERAM
- removed D1, D2, D3, D4, D5, D6, D7, D8: DIODE, DO-201AD_v
- removed D9: 3V3, DO-41_h
- removed LED1: led_enbl, LED_1206
- removed LED2: led_clk, LED_1206
- removed PIN1: pin_home, PIN_1x1-corn
- removed PIN10: osc_src, PIN_3x1
- removed PIN11: pin_enbl, PIN_1x1-corn
- removed PIN2: pin_ttl_pwr, PIN_2x1-corn
- removed PIN3: pin_drv_ctrl, PIN_3x1-corn
- removed PIN4: term_drv_pwr, DG300-5.0-02P-12
- removed PIN5: pin_switch_ctrl, PIN_3x1
- removed PIN6: pin_rst, PIN_1x1-corn
- removed PIN7: pin_sync, PIN_1x1-corn
- removed PIN8: term_out_ab, DG300-5.0-02P-12
- removed PIN9: term_out_cd, DG300-5.0-02P-12
- removed R1, R2: 470, RES_1206
- removed R3: 22k, RES_1206
- removed R4, R5: 0,5, R_5mm_hor
- removed R6: 47k, R_5mm_hor
- removed R8: 0, RES_1206
- removed U1: L297, DIP-20
- removed U2: L298N, multiwatt15v
Routing:
- net GND: track 208.4 -> 0.00 mm, vias 2 -> 0
- net +36V: track 131.2 -> 0.00 mm
- net N-000003: track 83.2 -> 0.00 mm
- net N-000008: track 82.6 -> 0.00 mm
- net N-0000025: track 80.4 -> 0.00 mm
- net N-0000026: track 29.3 -> 0.00 mm
