File: schematic/smdrv/mk1-rev5/sm-driver.kicad_pcb (KiCad board)
At the start: 2 copper layers, 35 parts, among them U1 L297, U2 L298N

Commit message: smdrv rev.5 pcb routing update
Parts:
- moved D5 193.8 mm to (298.0, 140.5), turned to 270 degrees
- moved D6 190.1 mm to (298.0, 126.0), turned to 270 degrees
- moved D1 186.6 mm to (290.5, 140.5), turned to 270 degrees
- moved PIN9 183.9 mm to (294.0, 114.0)
- moved D7 182.8 mm to (290.5, 126.0), turned to 270 degrees
- moved D2 181.6 mm to (283.0, 147.0), turned to 90 degrees
- moved D8 177.1 mm to (283.0, 132.5), turned to 90 degrees
- moved D4 175.0 mm to (276.0, 147.0), turned to 90 degrees
- moved PIN8 170.6 mm to (280.5, 114.0)
- moved D3 170.4 mm to (276.0, 132.5), turned to 90 degrees
- moved PIN4 156.8 mm to (266.5, 114.0)
- moved U2 156.7 mm to (257.0, 145.0), turned to 90 degrees
- moved PIN7 75.0 mm to (37.5, 84.5)
- moved PIN6 72.5 mm to (170.5, 41.0)
- moved PIN11 70.0 mm to (63.0, 134.0)
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Routing:
- net GND: track 0.00 -> 208.4 mm, vias 0 -> 2
- net +36V: track 0.00 -> 131.2 mm
- net N-000003: track 0.00 -> 83.2 mm
- net N-000008: track 0.00 -> 82.6 mm
- net N-0000025: track 0.00 -> 80.4 mm
- net N-0000026: track 0.00 -> 29.3 mm
Other:
- net class Default: trace_width 0.254 -> 0.3; via_dia 0.889 -> 1.2; via_drill 0.635 -> 0.8
- rule trace_min: 0.254 -> 0.3
- rule via_min_drill: 0.508 -> 0.8
- rule via_min_size: 0.889 -> 1.2
